File: hardware/Main board/_autosave-Main board.sch (KiCad schematic (older format))
At the start: 104 parts, among them J1 Wind Direction, J10 Free Pins, J11 Nokia 5110 LCD, J12 3v3 in, J2 Wind Speed, J3 USB_B_Micro, J4 Micro_SD_Card, J5 Sensor board connector, J6 230V AC IN, J7 ISP programmer, J8 SPI1, J9 SPI2, SW1 SW_Push, SW2 SW_SPST, SW3 SW_Push, SW4 SW_Push, SW5 Page Switch btn, U1 FT232RL, U2 MCP6042, U4 ATmega1284P-AU, U5 DS3231MZ, U6 ENC28J60, U7 USB6B1, U8 DRV5053, Y1 16MHZ

Commit message: Fixed multiple issues
Parts:
- gave numbers to parts that had none: 1
Changed lines of the file:
@@
 	8100 2500 9450 2500
 $Comp
-L Transistor_FET:IRLML6402 Q?
+L Transistor_FET:IRLML6402 Q1
 U 1 1 5D57A33C
 P 1700 5900
-F 0 "Q?" H 1906 5854 50  0000 L CNN
+F 0 "Q1" H 1906 5854 50  0000 L CNN
 F 1 "IRLML6402" H 1906 5945 50  0000 L CNN
 F 2 "Package_TO_SOT_SMD:SOT-23" H 1900 5825 50  0001 L CIN
