File: hardware/Main board/Main board.kicad_pcb (KiCad board)
At the start: 2 copper layers, 237.8 x 92.5 mm, 109 parts, among them J1 Wind Direction, J10 Free Pins, J11 Nokia 5110 LCD, J12 3v3 in, J2 Wind Speed, J3 USB_B_Micro, J4 Micro_SD_Card, J5 Sensor board connector, J6 230V AC IN, J7 ISP programmer, J8 SPI1, J9 SPI2, Q1 IRLML2060, SW1 SW_Push, SW2 SW_SPST, SW3 SW_Push, SW4 SW_Push, SW5 Page Switch btn, U1 FT232RL, U2 MCP6042, U4 ATmega1284P-AU, U5 DS3231MZ, U6 ENC28J60, U7 USB6B1, U8 DRV5053, Y1 16MHZ

Commit message: Fixed multiple things
Parts:
- added R32: 10k, Resistor_SMD:R_0805_2012Metric, F.Cu at (215.3, 51.9)
- added R35: 10k, Resistor_SMD:R_0805_2012Metric, F.Cu at (215.3, 54.9)
- added R36: 10k, Resistor_SMD:R_0805_2012Metric, F.Cu at (215.3, 49.0)
- moved J6 10.1 mm to (50.4, 116.4), turned to 0 degrees
- moved R31 2.66 mm to (137.4, 41.3)
- moved C23 2.50 mm to (140.0, 41.2)
- moved SW2 2.11 mm to (51.0, 99.2)
- moved C15 1.61 mm to (64.2, 107.6), turned to 90 degrees
Connections:
- J7 pad 2: SCK -> VCC
- J7 pad 3: RST -> SCK
- J7 pad 4: Net-(J7-Pad4) -> MOSI
- J7 pad 5: MOSI -> RST
- U1 pad 1: TXD -> RXD
- U1 pad 5: RXD -> TXD
- U8 pad 2: Net-(R31-Pad1) -> GND
- U8 pad 3: GND -> Net-(R31-Pad1)
Routing:
- net VCC: track 858.1 -> 893.3 mm, vias 6 -> 7
- net SCK: track 380.8 -> 395.3 mm, vias 2 -> 4
- net /SD_CS: track 77.9 -> 90.3 mm, vias 2 -> 4
- net MOSI: track 339.3 -> 348.5 mm, vias 1 -> 3
- net MISO: track 292.3 -> 298.5 mm
- net Net-(J6-Pad1): track 16.9 -> 20.4 mm
- net GND: track 102.3 -> 98.9 mm
- net PA2: track 55.9 -> 58.2 mm
- net /ETHER_CS: track 135.8 -> 134.2 mm
- net TXD: track 55.6 -> 56.8 mm
- net Net-(R31-Pad1): track 3.13 -> 4.00 mm
Other:
- board text added: "OFF"
- board text added: "ON"

Commit message: Fixed multiple issues
Parts:
- removed R32, R35, R36: 10k, Resistor_SMD:R_0805_2012Metric
- Q1: value IRLML2060 -> IRLML6402
- moved R11 4.56 mm to (117.3, 82.0), turned to 0 degrees
- moved Q1 2.19 mm to (117.2, 85.1), turned to 270 degrees
- moved R33 0.65 mm to (120.5, 83.1)
Connections:
- J7 pad 2: VCC -> Net-(J7-Pad2)
- Q1 pad 2: Net-(J11-Pad7) -> VCC
- Q1 pad 3: VCC -> Net-(J11-Pad7)
Routing:
- net VCC: track 893.3 -> 869.4 mm, vias 7 -> 6
- net /SD_CS: track 90.3 -> 78.2 mm, vias 4 -> 2
- net MOSI: track 348.5 -> 337.1 mm, vias 3 -> 1
- net MISO: track 298.5 -> 292.0 mm
- net Net-(J11-Pad7): track 5.37 -> 9.32 mm
- net Net-(Q1-Pad1): track 7.04 -> 4.43 mm
- net SCK: track 395.3 -> 396.6 mm
- net PD7: track 80.1 -> 79.4 mm
Other:
- board text added: "Motherboard for a weather station v1.1 by Daniels Fišers 19/08/2019"
- board text added: "Still no easter eggs here"
- board text removed: "Motherboard for a weather station v1 by Daniels Fišers 26/07/2019"
- board text removed: "No easter eggs here"

Commit message: Motherboard version v1.1
Parts:
- removed the REF** at (59.8, 109.2)
- added REF**: highVoltage, Meteo_Footprints:highVoltage, F.Cu at (60.0, 108.2)
- J4: footprint Connector_Card:microSD_HC_Hirose_DM3AT-SF-PEJM5 -> Meteo_Footprints:microSD
Connections:
- RV1 pad 3: GND -> dirOUT
- RV2 pad 3: GND -> Net-(R14-Pad2)
Routing:
- net dirOUT: track 30.2 -> 36.1 mm
- net Net-(R14-Pad2): track 3.42 -> 6.84 mm
