File: hardware/Main board/Main board.sch (KiCad schematic (older format))
At the start: 104 parts, among them J1 Wind Direction, J10 Free Pins, J11 Nokia 5110 LCD, J12 3v3 in, J2 Wind Speed, J3 USB_B_Micro, J4 Micro_SD_Card, J5 Sensor board connector, J6 230V AC IN, J7 ISP programmer, J8 SPI1, J9 SPI2, SW1 SW_Push, SW2 SW_SPST, SW3 SW_Push, SW4 SW_Push, SW5 Page Switch btn, U1 FT232RL, U2 MCP6042, U4 ATmega1284P-AU, U5 DS3231MZ, U6 ENC28J60, U7 USB6B1, U8 DRV5053, Y1 16MHZ

Commit message: Motherboard version v1.1
Parts:
- J4: footprint Connector_Card:microSD_HC_Hirose_DM3AT-SF-PEJM5 -> Meteo_Footprints:microSD
- gave numbers to parts that had none: 1
Connections:
- wire segments 217 -> 220
Changed lines of the file:
@@
 F 0 "J4" H 10300 3417 50  0000 C CNN
 F 1 "Micro_SD_Card" H 10300 3326 50  0000 C CNN
-F 2 "Connector_Card:microSD_HC_Hirose_DM3AT-SF-PEJM5" H 11500 3000 50  0001 C CNN
+F 2 "Meteo_Footprints:microSD" H 11500 3000 50  0001 C CNN
 F 3 "http://katalog.we-online.de/em/datasheet/693072010801.pdf" H 10350 2700 50  0001 C CNN
 	1    10350 2700
@@
 $EndComp
 $Comp
-L power:GND #PWR023
-U 1 1 5D37E5BC
-P 4650 2450
-F 0 "#PWR023" H 4650 2200 50  0001 C CNN
-F 1 "GND" H 4655 2277 50  0000 C CNN
-F 2 "" H 4650 2450 50  0001 C CNN
-F 3 "" H 4650 2450 50  0001 C CNN
-	1    4650 2450
-	1    0    0    -1
-$EndComp
-$Comp
 L power:GND #PWR021
 U 1 1 5D37ED58
@@
 $EndComp
 $Comp
-L power:GND #PWR014
-U 1 1 5D382912
-P 3100 1800
-F 0 "#PWR014" H 3100 1550 50  0001 C CNN
-F 1 "GND" V 3105 1672 50  0000 R CNN
-F 2 "" H 3100 1800 50  0001 C CNN
-F 3 "" H 3100 1800 50  0001 C CNN
-	1    3100 1800
-	0    -1   -1   0
-$EndComp
-$Comp
 L power:VCC #PWR07
 U 1 1 5D383503
@@
 	8100 2500 9450 2500
 $Comp
-L Transistor_FET:IRLML6402 Q?
+L Transistor_FET:IRLML6402 Q1
 U 1 1 5D57A33C
 P 1700 5900
-F 0 "Q?" H 1906 5854 50  0000 L CNN
+F 0 "Q1" H 1906 5854 50  0000 L CNN
 F 1 "IRLML6402" H 1906 5945 50  0000 L CNN
 F 2 "Package_TO_SOT_SMD:SOT-23" H 1900 5825 50  0001 L CIN
@@
 Wire Wire Line
 	1050 6400 1600 6400
+Wire Wire Line
+	3100 1800 3100 1650
+Wire Wire Line
+	4650 2450 4800 2450
+Wire Wire Line
+	4800 2450 4800 2300
+Connection ~ 4800 2300
 $EndSCHEMATC
